File: cad/PSU.kicad_pcb (KiCad board)
At the start: 2 copper layers, 15 parts, among them J1 Input, J2 INA219 breakout, J3 Output, J4 WWG-A, J5 WWG-B, Q1 LM317T, U1 LM7805_TO220, U3 X9C103P

Commit message: change wiring to make layout easier
Parts:
- moved R1 11.5 mm to (99.1, 90.2)
- moved U3 10.5 mm to (78.7, 91.4)
- moved D1 6.35 mm to (85.1, 83.8)
- moved C3 3.59 mm to (101.6, 83.8), turned to 0 degrees
- moved C1 2.54 mm to (102.9, 73.7)
- turned C4 to 270 degrees
Connections:
- J4 pad 5: Net-(J2-Pad4) -> Net-(J2-Pad3)
- J4 pad 6: Net-(J2-Pad3) -> Net-(J2-Pad4)
- U3 pad 1: Net-(J4-Pad7) -> Net-(J4-Pad3)
- U3 pad 2: Net-(J4-Pad3) -> Net-(J4-Pad7)
Routing:
- net +15V: track 0.00 -> 68.9 mm
- net Net-(C4-Pad1): track 0.00 -> 23.7 mm
- net Net-(C3-Pad1): track 0.00 -> 16.3 mm
Changed lines of the file:
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@@
     (thickness 1.6)
     (drawings 1)
-    (tracks 0)
+    (tracks 22)
     (zones 0)
     (modules 15)
@@
   )
   (module Diode_THT:D_DO-41_SOD81_P10.16mm_Horizontal (layer F.Cu)
-    (at 78.74 83.82)
+    (at 85.09 83.82)
     (descr "Diode, DO-41_SOD81 series, Axial, Horizontal, pin pitch=10.16mm, , length*diameter=5.2*2.7mm^2, , http://www.diodes.com/_files/packages/DO-41%20(Plastic).pdf")
     (tags "Diode DO-41_SOD81 series Axial Horizontal pin pitch 10.16mm  length 5.2mm diameter 2.7mm")
@@
   )
   (module Capacitor_THT:CP_Radial_D5.0mm_P2.00mm (layer F.Cu)
-    (at 102.87 71.12 90)
+    (at 102.87 73.66 90)
     (descr "CP, Radial series, Radial, pin pitch=2.00mm, , diameter=5mm, Electrolytic Capacitor")
     (tags "CP Radial series Radial pin pitch 2.00mm  diameter 5mm Electrolytic Capacitor")
@@
   )
   (module Capacitor_THT:CP_Radial_D5.0mm_P2.00mm (layer F.Cu)
-    (at 104.14 86.36 180)
+    (at 101.6 83.82)
     (descr "CP, Radial series, Radial, pin pitch=2.00mm, , diameter=5mm, Electrolytic Capacitor")
     (tags "CP Radial series Radial pin pitch 2.00mm  diameter 5mm Electrolytic Capacitor")
-    (fp_text reference C3 (at 1 -3.75 180) (layer F.SilkS)
-      (effects (font (size 1 1) (thickness 0.15)))
-    )
-    (fp_text value 47u (at 1 3.75 180) (layer F.Fab)
+    (fp_text reference C3 (at 1 -3.75) (layer F.SilkS)
+      (effects (font (size 1 1) (thickness 0.15)))
+    )
+    (fp_text value 47u (at 1 3.75) (layer F.Fab)
       (effects (font (size 1 1) (thickness 0.15)))
     )
@@
     (fp_line (start -1.804775 -1.475) (end -1.304775 -1.475) (layer F.SilkS) (width 0.12))
     (fp_line (start -1.554775 -1.725) (end -1.554775 -1.225) (layer F.SilkS) (width 0.12))
-    (fp_text user %R (at 1 0 180) (layer F.Fab)
-      (effects (font (size 1 1) (thickness 0.15)))
-    )
-    (pad 1 thru_hole rect (at 0 0 180) (size 1.6 1.6) (drill 0.8) (layers *.Cu *.Mask)
+    (fp_text user %R (at 1 0) (layer F.Fab)
+      (effects (font (size 1 1) (thickness 0.15)))
+    )
+    (pad 1 thru_hole rect (at 0 0) (size 1.6 1.6) (drill 0.8) (layers *.Cu *.Mask)
       (net 3 "Net-(C3-Pad1)"))
-    (pad 2 thru_hole circle (at 2 0 180) (size 1.6 1.6) (drill 0.8) (layers *.Cu *.Mask)
+    (pad 2 thru_hole circle (at 2 0) (size 1.6 1.6) (drill 0.8) (layers *.Cu *.Mask)
       (net 1 GND))
     (model ${KISYS3DMOD}/Capacitor_THT.3dshapes/CP_Radial_D5.0mm_P2.00mm.wrl
@@
   )
   (module Capacitor_THT:CP_Radial_D6.3mm_P2.50mm (layer F.Cu)
-    (at 83.82 69.85 180)
+    (at 83.82 69.85 270)
     (descr "CP, Radial series, Radial, pin pitch=2.50mm, , diameter=6.3mm, Electrolytic Capacitor")
     (tags "CP Radial series Radial pin pitch 2.50mm  diameter 6.3mm Electrolytic Capacitor")
-    (fp_text reference C4 (at 1.25 -4.4 180) (layer F.SilkS)
-      (effects (font (size 1 1) (thickness 0.15)))
-    )
-    (fp_text value 220u (at 1.25 4.4 180) (layer F.Fab)
+    (fp_text reference C4 (at 1.25 -4.4 270) (layer F.SilkS)
+      (effects (font (size 1 1) (thickness 0.15)))
+    )
+    (fp_text value 220u (at 1.25 4.4 270) (layer F.Fab)
       (effects (font (size 1 1) (thickness 0.15)))
     )
@@
     (fp_line (start -2.250241 -1.839) (end -1.620241 -1.839) (layer F.SilkS) (width 0.12))
     (fp_line (start -1.935241 -2.154) (end -1.935241 -1.524) (layer F.SilkS) (width 0.12))
-    (fp_text user %R (at 1.25 0 180) (layer F.Fab)
-      (effects (font (size 1 1) (thickness 0.15)))
-    )
-    (pad 1 thru_hole rect (at 0 0 180) (size 1.6 1.6) (drill 0.8) (layers *.Cu *.Mask)
+    (fp_text user %R (at 1.25 0 270) (layer F.Fab)
+      (effects (font (size 1 1) (thickness 0.15)))
+    )
+    (pad 1 thru_hole rect (at 0 0 270) (size 1.6 1.6) (drill 0.8) (layers *.Cu *.Mask)
       (net 4 "Net-(C4-Pad1)"))
-    (pad 2 thru_hole circle (at 2.5 0 180) (size 1.6 1.6) (drill 0.8) (layers *.Cu *.Mask)
+    (pad 2 thru_hole circle (at 2.5 0 270) (size 1.6 1.6) (drill 0.8) (layers *.Cu *.Mask)
       (net 1 GND))
     (model ${KISYS3DMOD}/Capacitor_THT.3dshapes/CP_Radial_D6.3mm_P2.50mm.wrl
@@
       (net 10 "Net-(J4-Pad4)"))
     (pad 5 thru_hole oval (at 0 10.16) (size 1.7 1.7) (drill 1) (layers *.Cu *.Mask)
+      (net 6 "Net-(J2-Pad3)"))
+    (pad 6 thru_hole oval (at 0 12.7) (size 1.7 1.7) (drill 1) (layers *.Cu *.Mask)
       (net 7 "Net-(J2-Pad4)"))
-    (pad 6 thru_hole oval (at 0 12.7) (size 1.7 1.7) (drill 1) (layers *.Cu *.Mask)
-      (net 6 "Net-(J2-Pad3)"))
     (pad 7 thru_hole oval (at 0 15.24) (size 1.7 1.7) (drill 1) (layers *.Cu *.Mask)
       (net 11 "Net-(J4-Pad7)"))
@@
   )
   (module Resistor_THT:R_Axial_DIN0207_L6.3mm_D2.5mm_P7.62mm_Horizontal (layer F.Cu)
-    (at 87.63 91.44 180)
+    (at 99.06 90.17 180)
     (descr "Resistor, Axial_DIN0207 series, Axial, Horizontal, pin pitch=7.62mm, 0.25W = 1/4W, length*diameter=6.3*2.5mm^2, http://cdn-reichelt.de/documents/datenblatt/B400/1_4W%23YAG.pdf")
     (tags "Resistor Axial_DIN0207 series Axial Horizontal pin pitch 7.62mm 0.25W = 1/4W length 6.3mm diameter 2.5mm")
@@
   )
   (module X9C103P:DIP254P762X533-8 (layer F.Cu)
-    (at 68.58 93.98)
+    (at 78.74 91.44)
     (fp_text reference U3 (at -4.01713 -11.848) (layer F.SilkS)
       (effects (font (size 1.64161 1.64161) (thickness 0.05)))
@@
     (fp_arc (start -3.81 -8.89) (end -4.1148 -8.89) (angle -180) (layer Eco2.User) (width 0))
     (pad 1 thru_hole rect (at -7.62 -7.62) (size 1.6764 1.6764) (drill 1.1176) (layers *.Cu *.Mask)
+      (net 9 "Net-(J4-Pad3)"))
+    (pad 2 thru_hole circle (at -7.62 -5.08) (size 1.6764 1.6764) (drill 1.1176) (layers *.Cu *.Mask)
       (net 11 "Net-(J4-Pad7)"))
-    (pad 2 thru_hole circle (at -7.62 -5.08) (size 1.6764 1.6764) (drill 1.1176) (layers *.Cu *.Mask)
-      (net 9 "Net-(J4-Pad3)"))
     (pad 3 thru_hole circle (at -7.62 -2.54) (size 1.6764 1.6764) (drill 1.1176) (layers *.Cu *.Mask)
       (net 22 "Net-(U3-Pad3)"))
@@
     (arrow2b (pts (xy 80.01 132.08) (xy 81.136504 131.493579)))
   )
+  (segment (start 119.38 82.5975) (end 113.0775 88.9) (width 0.25) (layer F.Cu) (net 2))
+  (segment (start 119.38 69.85) (end 119.38 82.5975) (width 0.25) (layer F.Cu) (net 2))
+  (segment (start 114.02 73.66) (end 103.92 73.66) (width 0.25) (layer F.Cu) (net 2))
+  (segment (start 103.92 73.66) (end 102.87 73.66) (width 0.25) (layer F.Cu) (net 2))
+  (segment (start 117.83 69.85) (end 114.02 73.66) (width 0.25) (layer F.Cu) (net 2))
+  (segment (start 119.38 69.85) (end 117.83 69.85) (width 0.25) (layer F.Cu) (net 2))
+  (segment (start 102.87 73.66) (end 93.98 73.66) (width 0.25) (layer F.Cu) (net 2))
+  (segment (start 102.8025 97.79) (end 101.6 97.79) (width 0.25) (layer F.Cu) (net 2))
+  (segment (start 114.35501 94.509161) (end 111.074171 97.79) (width 0.25) (layer F.Cu) (net 2))
+  (segment (start 111.074171 97.79) (end 102.8025 97.79) (width 0.25) (layer F.Cu) (net 2))
+  (segment (start 114.35501 90.17751) (end 114.35501 94.509161) (width 0.25) (layer F.Cu) (net 2))
+  (segment (start 113.0775 88.9) (end 114.35501 90.17751) (width 0.25) (layer F.Cu) (net 2))
+  (segment (start 113.03 88.9) (end 113.0775 88.9) (width 0.25) (layer F.Cu) (net 2))
+  (segment (start 101.6 84.87) (end 101.6 83.82) (width 0.25) (layer F.Cu) (net 3))
+  (segment (start 110.71 93.98) (end 101.6 84.87) (width 0.25) (layer F.Cu) (net 3))
+  (segment (start 113.03 93.98) (end 110.71 93.98) (width 0.25) (layer F.Cu) (net 3))
+  (segment (start 74.93 66.12) (end 74.93 64.77) (width 0.25) (layer F.Cu) (net 4))
+  (segment (start 78.66 69.85) (end 74.93 66.12) (width 0.25) (layer F.Cu) (net 4))
+  (segment (start 83.82 69.85) (end 78.66 69.85) (width 0.25) (layer F.Cu) (net 4))
+  (segment (start 69.57 64.77) (end 66.04 68.3) (width 0.25) (layer F.Cu) (net 4))
+  (segment (start 66.04 68.3) (end 66.04 69.85) (width 0.25) (layer F.Cu) (net 4))
+  (segment (start 74.93 64.77) (end 69.57 64.77) (width 0.25) (layer F.Cu) (net 4))
 )

Commit message: more pcb
Routing:
- net Net-(J2-Pad5): track 0.00 -> 71.7 mm, vias 0 -> 1
- net Net-(C4-Pad1): track 23.7 -> 77.3 mm
- net Net-(J5-Pad6): track 0.00 -> 53.0 mm, vias 0 -> 1
- net Net-(J4-Pad7): track 0.00 -> 43.9 mm
- net +5V: track 0.00 -> 42.8 mm
- net Net-(J4-Pad3): track 0.00 -> 37.9 mm
- net Net-(Q1-Pad1): track 0.00 -> 23.0 mm
- net Net-(J2-Pad4): track 0.00 -> 12.3 mm
- net Net-(J2-Pad3): track 0.00 -> 12.3 mm
- net Net-(C3-Pad1): track 16.3 -> 22.6 mm
- net GND: track 0.00 -> 3.69 mm
- net +15V: track 68.9 -> 71.8 mm
- added copper zone on B.Cu, net GND
Other:
- net class Power added: clearance 0.3, trace_width 0.5, via_dia 1, via_drill 0.6
Changed lines of the file:
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@@
     (thickness 1.6)
     (drawings 1)
-    (tracks 22)
+    (tracks 72)
     (zones 0)
     (modules 15)
@@
     (uvia_dia 0.3)
     (uvia_drill 0.1)
-    (add_net +15V)
-    (add_net +5V)
-    (add_net GND)
     (add_net "Net-(C3-Pad1)")
-    (add_net "Net-(C4-Pad1)")
     (add_net "Net-(J2-Pad3)")
     (add_net "Net-(J2-Pad4)")
-    (add_net "Net-(J2-Pad5)")
     (add_net "Net-(J4-Pad3)")
     (add_net "Net-(J4-Pad4)")
@@
     (add_net "Net-(Q1-Pad1)")
     (add_net "Net-(U3-Pad3)")
+  )
+  (net_class Power ""
+    (clearance 0.3)
+    (trace_width 0.5)
+    (via_dia 1)
+    (via_drill 0.6)
+    (uvia_dia 0.3)
+    (uvia_drill 0.1)
+    (add_net +15V)
+    (add_net +5V)
+    (add_net GND)
+    (add_net "Net-(C4-Pad1)")
+    (add_net "Net-(J2-Pad5)")
   )
   (module Diode_THT:D_DO-41_SOD81_P10.16mm_Horizontal (layer F.Cu)
@@
     (arrow2b (pts (xy 80.01 132.08) (xy 81.136504 131.493579)))
   )
-  (segment (start 119.38 82.5975) (end 113.0775 88.9) (width 0.25) (layer F.Cu) (net 2))
-  (segment (start 119.38 69.85) (end 119.38 82.5975) (width 0.25) (layer F.Cu) (net 2))
-  (segment (start 114.02 73.66) (end 103.92 73.66) (width 0.25) (layer F.Cu) (net 2))
-  (segment (start 103.92 73.66) (end 102.87 73.66) (width 0.25) (layer F.Cu) (net 2))
-  (segment (start 117.83 69.85) (end 114.02 73.66) (width 0.25) (layer F.Cu) (net 2))
+  (segment (start 114.38 69.85) (end 112.57 71.66) (width 0.25) (layer F.Cu) (net 1))
+  (segment (start 103.6 82.68863) (end 103.6 83.82) (width 0.25) (layer B.Cu) (net 1))
+  (segment (start 119.38 82.5975) (end 113.0775 88.9) (width 0.5) (layer F.Cu) (net 2))
+  (segment (start 119.38 69.85) (end 119.38 82.5975) (width 0.5) (layer F.Cu) (net 2))
+  (segment (start 117.83 69.85) (end 114.02 73.66) (width 0.5) (layer F.Cu) (net 2))
   (segment (start 119.38 69.85) (end 117.83 69.85) (width 0.25) (layer F.Cu) (net 2))
-  (segment (start 102.87 73.66) (end 93.98 73.66) (width 0.25) (layer F.Cu) (net 2))
+  (segment (start 102.87 73.66) (end 93.98 73.66) (width 0.5) (layer F.Cu) (net 2))
   (segment (start 102.8025 97.79) (end 101.6 97.79) (width 0.25) (layer F.Cu) (net 2))
-  (segment (start 114.35501 94.509161) (end 111.074171 97.79) (width 0.25) (layer F.Cu) (net 2))
-  (segment (start 111.074171 97.79) (end 102.8025 97.79) (width 0.25) (layer F.Cu) (net 2))
-  (segment (start 114.35501 90.17751) (end 114.35501 94.509161) (width 0.25) (layer F.Cu) (net 2))
-  (segment (start 113.0775 88.9) (end 114.35501 90.17751) (width 0.25) (layer F.Cu) (net 2))
-  (segment (start 113.03 88.9) (end 113.0775 88.9) (width 0.25) (layer F.Cu) (net 2))
+  (segment (start 111.074171 97.79) (end 102.8025 97.79) (width 0.5) (layer F.Cu) (net 2))
+  (segment (start 114.02 73.66) (end 102.87 73.66) (width 0.5) (layer F.Cu) (net 2))
+  (segment (start 111.074171 97.79) (end 114.3 97.79) (width 0.5) (layer F.Cu) (net 2))
+  (segment (start 114.3 97.79) (end 115.57 96.52) (width 0.5) (layer F.Cu) (net 2))
+  (segment (start 113.0775 88.9) (end 113.03 88.9) (width 0.5) (layer F.Cu) (net 2))
+  (segment (start 115.57 91.3925) (end 113.0775 88.9) (width 0.5) (layer F.Cu) (net 2))
+  (segment (start 115.57 96.52) (end 115.57 91.3925) (width 0.5) (layer F.Cu) (net 2))
   (segment (start 101.6 84.87) (end 101.6 83.82) (width 0.25) (layer F.Cu) (net 3))
   (segment (start 110.71 93.98) (end 101.6 84.87) (width 0.25) (layer F.Cu) (net 3))
   (segment (start 113.03 93.98) (end 110.71 93.98) (width 0.25) (layer F.Cu) (net 3))
+  (segment (start 95.25 83.82) (end 101.6 83.82) (width 0.25) (layer F.Cu) (net 3))
   (segment (start 74.93 66.12) (end 74.93 64.77) (width 0.25) (layer F.Cu) (net 4))
   (segment (start 78.66 69.85) (end 74.93 66.12) (width 0.25) (layer F.Cu) (net 4))
@@
   (segment (start 66.04 68.3) (end 66.04 69.85) (width 0.25) (layer F.Cu) (net 4))
   (segment (start 74.93 64.77) (end 69.57 64.77) (width 0.25) (layer F.Cu) (net 4))
+  (segment (start 66.04 118.11) (end 69.85 121.92) (width 0.5) (layer B.Cu) (net 4))
+  (segment (start 66.04 69.85) (end 66.04 118.11) (width 0.5) (layer B.Cu) (net 4))
+  (segment (start 78.74 83.82) (end 85.09 83.82) (width 0.5) (layer F.Cu) (net 5))
+  (segment (start 79.578199 84.658199) (end 78.74 83.82) (width 0.25) (layer B.Cu) (net 5))
+  (segment (start 80.46001 85.54001) (end 79.578199 84.658199) (width 0.5) (layer B.Cu) (net 5))
+  (segment (start 80.46001 107.66999) (end 80.46001 85.54001) (width 0.5) (layer B.Cu) (net 5))
+  (segment (start 80.01 108.12) (end 80.46001 107.66999) (width 0.5) (layer B.Cu) (net 5))
+  (segment (start 80.01 109.22) (end 80.01 108.12) (width 0.25) (layer B.Cu) (net 5))
+  (segment (start 80.01 109.22) (end 69.85 109.22) (width 0.5) (layer F.Cu) (net 5))
+  (segment (start 74.93 114.3) (end 80.01 119.38) (width 0.25) (layer F.Cu) (net 6))
+  (segment (start 69.85 114.3) (end 74.93 114.3) (width 0.25) (layer F.Cu) (net 6))
+  (segment (start 74.93 116.84) (end 80.01 121.92) (width 0.25) (layer F.Cu) (net 7))
+  (segment (start 69.85 116.84) (end 74.93 116.84) (width 0.25) (layer F.Cu) (net 7))
+  (segment (start 99.06 90.17) (end 99.06 97.79) (width 0.5) (layer F.Cu) (net 8))
+  (segment (start 99.06 97.8375) (end 99.06 97.79) (width 0.25) (layer F.Cu) (net 8))
+  (segment (start 69.85 119.38) (end 72.39 119.38) (width 0.5) (layer B.Cu) (net 8))
+  (segment (start 72.39 119.38) (end 72.39 128.27) (width 0.5) (layer B.Cu) (net 8))
+  (segment (start 72.39 128.27) (end 74.93 130.81) (width 0.5) (layer B.Cu) (net 8))
+  (segment (start 74.93 130.81) (end 85.09 130.81) (width 0.5) (layer B.Cu) (net 8))
+  (segment (start 85.09 130.81) (end 85.09 121.92) (width 0.5) (layer B.Cu) (net 8))
+  (segment (start 85.09 121.92) (end 97.79 109.22) (width 0.5) (layer B.Cu) (net 8))
+  (segment (start 97.79 109.22) (end 97.79 109.22) (width 0.5) (layer B.Cu) (net 8))
+  (via (at 97.79 109.22) (size 1) (drill 0.6) (layers F.Cu B.Cu) (net 8))
+  (segment (start 99.06 97.79) (end 99.06 107.95) (width 0.5) (layer F.Cu) (net 8))
+  (segment (start 99.06 107.95) (end 97.79 109.22) (width 0.5) (layer F.Cu) (net 8))
+  (segment (start 79.160001 113.450001) (end 80.01 114.3) (width 0.25) (layer B.Cu) (net 9))
+  (segment (start 71.12 83.82) (end 72.2082 83.82) (width 0.25) (layer B.Cu) (net 9))
+  (segment (start 71.12 83.82) (end 73.66 83.82) (width 0.25) (layer B.Cu) (net 9))
+  (segment (start 73.66 83.82) (end 76.2 86.36) (width 0.25) (layer B.Cu) (net 9))
+  (segment (start 76.2 110.49) (end 80.01 114.3) (width 0.25) (layer B.Cu) (net 9))
+  (segment (start 76.2 86.36) (end 76.2 110.49) (width 0.25) (layer B.Cu) (net 9))
+  (segment (start 68.58 88.9) (end 68.58 99.06) (width 0.25) (layer B.Cu) (net 11))
+  (segment (start 71.12 86.36) (end 68.58 88.9) (width 0.25) (layer B.Cu) (net 11))
+  (segment (start 68.58 99.06) (end 73.66 104.14) (width 0.25) (layer B.Cu) (net 11))
+  (segment (start 73.66 118.11) (end 80.01 124.46) (width 0.25) (layer B.Cu) (net 11))
+  (segment (start 73.66 104.14) (end 73.66 118.11) (width 0.25) (layer B.Cu) (net 11))
+  (segment (start 115.57 121.92) (end 84.356501 90.706501) (width 0.25) (layer B.Cu) (net 15))
+  (segment (start 78.74 86.36) (end 82.55 86.36) (width 0.25) (layer F.Cu) (net 15))
+  (segment (start 82.55 86.36) (end 82.55 86.36) (width 0.25) (layer F.Cu) (net 15))
+  (via (at 82.55 86.36) (size 0.8) (drill 0.4) (layers F.Cu B.Cu) (net 15))
+  (segment (start 84.356501 88.166501) (end 82.55 86.36) (width 0.25) (layer B.Cu) (net 15))
+  (segment (start 84.356501 90.706501) (end 84.356501 88.166501) (width 0.25) (layer B.Cu) (net 15))
+  (segment (start 90.17 91.44) (end 91.44 90.17) (width 0.25) (layer F.Cu) (net 21))
+  (segment (start 78.74 91.44) (end 90.17 91.44) (width 0.25) (layer F.Cu) (net 21))
+  (segment (start 90.17 91.44) (end 90.17 92.71) (width 0.25) (layer F.Cu) (net 21))
+  (segment (start 95.25 97.79) (end 96.52 97.79) (width 0.25) (layer F.Cu) (net 21))
+  (segment (start 90.17 92.71) (end 95.25 97.79) (width 0.25) (layer F.Cu) (net 21))
+  (zone (net 1) (net_name GND) (layer B.Cu) (hatch edge 0.508)
+    (connect_pads (clearance 0.508))
+    (min_thickness 0.254)
+    (fill yes (arc_segments 16) (thermal_gap 0.508) (thermal_bridge_width 0.508))
+    (polygon
+      (pts
+        (xy 55.88 62.23) (xy 124.46 62.23) (xy 124.46 135.89) (xy 55.88 135.89)
+      )
+    )
+  )
 )

Commit message: add barrel jack and layout pcb again
Parts:
- removed U3: X9C103P, X9C103P:DIP254P762X533-8
- added J6: WWG-B, Connector_PinHeader_2.54mm:PinHeader_1x08_P2.54mm_Vertical, F.Cu at (116.8, 68.6)
- added REF**: MountingHole_2.7mm_M2.5_Pad, MountingHole:MountingHole_2.7mm_M2.5_Pad, F.Cu at (43.2, 90.2)
- added REF**: MountingHole_2.7mm_M2.5_Pad, MountingHole:MountingHole_2.7mm_M2.5_Pad, F.Cu at (127.0, 90.2)
- added REF**: MountingHole_2.7mm_M2.5_Pad, MountingHole:MountingHole_2.7mm_M2.5_Pad, F.Cu at (127.0, 36.8)
- added REF**: MountingHole_2.7mm_M2.5_Pad, MountingHole:MountingHole_2.7mm_M2.5_Pad, F.Cu at (43.2, 36.8)
- added U2: X9C103P, X9C103P:DIP254P762X533-8, F.Cu at (102.9, 86.4)
- J2: value INA219 breakout -> Barrel_Jack_Switch; footprint Connector_PinHeader_2.54mm:PinHeader_1x06_P2.54mm_Vertical -> Connector_BarrelJack:BarrelJack_CUI_PJ-102AH_Horizontal
- J4: value WWG-A -> INA219 breakout; footprint Connector_PinHeader_2.54mm:PinHeader_1x08_P2.54mm_Vertical -> Connector_PinHeader_2.54mm:PinHeader_1x06_P2.54mm_Vertical
- J5: value WWG-B -> WWG-A
- moved J1 65.5 mm to (57.1, 49.5)
- moved U1 61.9 mm to (54.6, 68.6), turned to 90 degrees
- moved J3 60.7 mm to (124.5, 53.3), turned to 90 degrees
- moved J4 60.7 mm to (100.3, 52.1), turned to 270 degrees
- moved J5 53.2 mm to (81.3, 68.6)
- moved Q1 52.9 mm to (69.8, 52.1)
- moved C1 44.7 mm to (59.7, 85.1), turned to 270 degrees
- moved R1 39.5 mm to (77.5, 57.1)
- moved C3 37.0 mm to (67.3, 69.8), turned to 270 degrees
- moved C2 34.9 mm to (59.7, 80.0)
- moved C4 34.9 mm to (113.0, 50.8), turned to 90 degrees
- moved J2 31.0 mm to (52.1, 83.8), turned to 270 degrees
- moved D1 23.3 mm to (73.7, 63.5), turned to 180 degrees
- moved D2 14.8 mm to (87.6, 57.1), turned to 0 degrees
Connections:
- J2 pad 1: +5V -> +15V
- J2 pad 3: Net-(J2-Pad3) -> GND
- J4 pad 5: Net-(J2-Pad3) -> Net-(J4-Pad5)
- J4 pad 6: Net-(J2-Pad4) -> Net-(C4-Pad1)
- J5 pad 1: Net-(J5-Pad1) -> +5V
- J5 pad 2: Net-(J5-Pad2) -> GND
- J5 pad 5: Net-(J5-Pad5) -> Net-(J4-Pad4)
- J5 pad 6: Net-(J5-Pad6) -> Net-(J4-Pad3)
- Q1 pad 2: Net-(J2-Pad5) -> Net-(J4-Pad5)
- R1 pad 1: Net-(J2-Pad5) -> Net-(J4-Pad5)
Routing:
- net GND: track 3.69 -> 179.7 mm
- net Net-(J2-Pad5): track 71.7 -> 0.00 mm, vias 1 -> 0
- net Net-(J5-Pad6): track 53.0 -> 0.00 mm, vias 1 -> 0
- net +5V: track 42.8 -> 92.2 mm
- net Net-(Q1-Pad1): track 23.0 -> 70.5 mm
- net Net-(J4-Pad7): track 43.9 -> 0.00 mm
- net Net-(C4-Pad1): track 77.3 -> 45.8 mm
- net Net-(J4-Pad4): track 0.00 -> 31.4 mm
- net Net-(J4-Pad5): track 0.00 -> 28.6 mm
- net Net-(J5-Pad3): track 0.00 -> 16.1 mm
- net Net-(J5-Pad7): track 0.00 -> 15.0 mm
- net Net-(J6-Pad6): track 0.00 -> 14.0 mm
- net Net-(J2-Pad4): track 12.3 -> 0.00 mm
- net Net-(J2-Pad3): track 12.3 -> 0.00 mm
- net Net-(C3-Pad1): track 22.6 -> 17.4 mm
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Other:
- board outline added: 94 x 63.5 mm
- net class +15V added: clearance 0.2, trace_width 0.5, via_dia 0.8, via_drill 0.4
- net class +5V added: clearance 0.2, trace_width 0.5, via_dia 0.8, via_drill 0.4
- net class GND added: clearance 0.2, trace_width 0.5, via_dia 0.8, via_drill 0.4
- net class Power removed
- rule pad_to_mask_clearance: 0.051 -> 0
- board text added: "PSU v1.0 (c) 2019 Steve"
- board text added: "heatsink"
