File: cad/PSU.sch (KiCad schematic (older format))
At the start: 15 parts, among them J1 Input, J2 INA219 breakout, J3 Output, J4 WWG-A, J5 WWG-B, U1 L7805, U2 LM317_3PinPackage, U3 X9C103P

Commit message: footprints
Parts:
- removed U1: L7805, symbol Regulator_Linear:L7805
- removed U2: LM317_3PinPackage, symbol Regulator_Linear:LM317_3PinPackage
- added Q1: LM317T, Package_TO_SOT_THT:TO-220-3_Vertical, symbol LM317T:LM317T
- added U1: LM7805_TO220, Package_TO_SOT_THT:TO-220-3_Vertical, symbol Regulator_Linear:LM7805_TO220
- C1, C3: footprint (none) -> Capacitor_THT:CP_Radial_D5.0mm_P2.00mm
- C2: footprint (none) -> Capacitor_THT:C_Disc_D5.0mm_W2.5mm_P5.00mm
- C4: value 47u -> 220u; footprint (none) -> Capacitor_THT:CP_Radial_D6.3mm_P2.50mm
- D1, D2: footprint DO41-10 -> Diode_THT:D_A-405_P10.16mm_Horizontal
- J1, J3: footprint (none) -> TerminalBlock_Phoenix:TerminalBlock_Phoenix_PT-1,5-2-5.0-H_1x02_P5.00mm_Horizontal
- J2: footprint (none) -> Connector_PinHeader_2.54mm:PinHeader_1x06_P2.54mm_Vertical
- J4, J5: footprint (none) -> Connector_PinHeader_2.54mm:PinHeader_1x08_P2.54mm_Vertical
- R1: footprint (none) -> Resistor_THT:R_Axial_DIN0207_L6.3mm_D2.5mm_P7.62mm_Horizontal
Connections:
- wire segments 64 -> 67
Other:
- moved on the sheet: C1, C2, C3, C4, D1, D2, J1, J2, J3, J4, J5, R1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

Commit message: erc check
Connections:
- wire segments 67 -> 69
- no-connect marks 0 -> 10
Changed lines of the file:
@@
 L power:+15V #PWR0107
 U 1 1 5CD98A23
-P 2500 4150
-F 0 "#PWR0107" H 2500 4000 50  0001 C CNN
-F 1 "+15V" H 2515 4323 50  0000 C CNN
-F 2 "" H 2500 4150 50  0001 C CNN
-F 3 "" H 2500 4150 50  0001 C CNN
-	1    2500 4150
+P 2650 4150
+F 0 "#PWR0107" H 2650 4000 50  0001 C CNN
+F 1 "+15V" H 2665 4323 50  0000 C CNN
+F 2 "" H 2650 4150 50  0001 C CNN
+F 3 "" H 2650 4150 50  0001 C CNN
+	1    2650 4150
 	1    0    0    -1
 $EndComp
@@
 L power:GND #PWR0108
 U 1 1 5CD98A46
-P 2500 4250
-F 0 "#PWR0108" H 2500 4000 50  0001 C CNN
-F 1 "GND" H 2505 4077 50  0000 C CNN
-F 2 "" H 2500 4250 50  0001 C CNN
-F 3 "" H 2500 4250 50  0001 C CNN
-	1    2500 4250
+P 2650 4250
+F 0 "#PWR0108" H 2650 4000 50  0001 C CNN
+F 1 "GND" H 2655 4077 50  0000 C CNN
+F 2 "" H 2650 4250 50  0001 C CNN
+F 3 "" H 2650 4250 50  0001 C CNN
+	1    2650 4250
 	1    0    0    -1
 $EndComp
@@
 Wire Wire Line
 	4650 4450 4650 5150
+$Comp
+L power:PWR_FLAG #FLG0101
+U 1 1 5CE68781
+P 4400 2650
+F 0 "#FLG0101" H 4400 2725 50  0001 C CNN
+F 1 "PWR_FLAG" H 4400 2824 50  0001 C CNN
+F 2 "" H 4400 2650 50  0001 C CNN
+F 3 "~" H 4400 2650 50  0001 C CNN
+	1    4400 2650
+	1    0    0    -1
+$EndComp
+Connection ~ 4400 2650
+Wire Wire Line
+	2500 4150 2650 4150
+Wire Wire Line
+	2500 4250 2650 4250
+$Comp
+L power:PWR_FLAG #FLG0102
+U 1 1 5CE6B5B3
+P 2500 4150
+F 0 "#FLG0102" H 2500 4225 50  0001 C CNN
+F 1 "PWR_FLAG" H 2500 4324 50  0001 C CNN
+F 2 "" H 2500 4150 50  0001 C CNN
+F 3 "~" H 2500 4150 50  0001 C CNN
+	1    2500 4150
+	1    0    0    -1
+$EndComp
+Connection ~ 2500 4150
+$Comp
+L power:PWR_FLAG #FLG0103
+U 1 1 5CE6B602
+P 2500 4250
+F 0 "#FLG0103" H 2500 4325 50  0001 C CNN
+F 1 "PWR_FLAG" H 2500 4423 50  0001 C CNN
+F 2 "" H 2500 4250 50  0001 C CNN
+F 3 "~" H 2500 4250 50  0001 C CNN
+	1    2500 4250
+	1    0    0    1
+$EndComp
+Connection ~ 2500 4250
+NoConn ~ 8000 3200
+NoConn ~ 8000 3300
+NoConn ~ 8000 3400
+NoConn ~ 8000 3500
+NoConn ~ 8000 3600
+NoConn ~ 8000 3800
+NoConn ~ 8000 3900
+NoConn ~ 7200 3900
+NoConn ~ 7200 3500
+NoConn ~ 5000 5050
 $EndSCHEMATC

Commit message: first layout
Parts:
- removed D1, D2: 1N4001, Diode_THT:D_A-405_P10.16mm_Horizontal, symbol 1N4001:1N4001
- added D1, D2: 1N4001, Diode_THT:D_DO-41_SOD81_P10.16mm_Horizontal, symbol Diode:1N4001
Changed lines of the file:
@@
 Wire Wire Line
 	7150 3200 7200 3200
-$Comp
-L 1N4001:1N4001 D1
-U 1 1 5CE165D2
-P 4200 2650
-F 0 "D1" H 4250 2775 50  0000 C CNN
-F 1 "1N4001" H 4200 2650 50  0001 L BNN
-F 2 "Diode_THT:D_A-405_P10.16mm_Horizontal" H 4200 2650 50  0001 L BNN
-F 3 "ON Semiconductor" H 4200 2650 50  0001 L BNN
-F 4 "None" H 4200 2650 50  0001 L BNN "Field4"
-F 5 "DO-41 ON Semiconductor" H 4200 2650 50  0001 L BNN "Field5"
-F 6 "Unavailable" H 4200 2650 50  0001 L BNN "Field6"
-F 7 "1N4001" H 4200 2650 50  0001 L BNN "Field7"
-F 8 "Diode, Standard, 1A, 50V" H 4200 2650 50  0001 L BNN "Field8"
-	1    4200 2650
-	1    0    0    -1
-$EndComp
 Wire Wire Line
 	3900 2650 4100 2650
@@
 Wire Wire Line
 	5500 4000 5500 4250
-Wire Wire Line
-	5500 4000 5700 4000
 Wire Wire Line
 	5500 4350 5700 4350
@@
 $EndComp
 Connection ~ 6000 4000
-$Comp
-L 1N4001:1N4001 D2
-U 1 1 5CE1E838
-P 5700 4200
-F 0 "D2" V 5750 4120 50  0000 R CNN
-F 1 "1N4001" H 5700 4200 50  0001 L BNN
-F 2 "Diode_THT:D_A-405_P10.16mm_Horizontal" H 5700 4200 50  0001 L BNN
-F 3 "ON Semiconductor" H 5700 4200 50  0001 L BNN
-F 4 "None" H 5700 4200 50  0001 L BNN "Field4"
-F 5 "DO-41 ON Semiconductor" H 5700 4200 50  0001 L BNN "Field5"
-F 6 "Unavailable" H 5700 4200 50  0001 L BNN "Field6"
-F 7 "1N4001" H 5700 4200 50  0001 L BNN "Field7"
-F 8 "Diode, Standard, 1A, 50V" H 5700 4200 50  0001 L BNN "Field8"
-	1    5700 4200
-	0    -1   -1   0
-$EndComp
-Connection ~ 5700 4000
-Wire Wire Line
-	5700 4000 6000 4000
 Wire Wire Line
 	6000 4300 6000 4350
@@
 	1    0    0    -1
 $EndComp
-Connection ~ 4400 2650
 Wire Wire Line
 	2500 4150 2650 4150
@@
 NoConn ~ 7200 3500
 NoConn ~ 5000 5050
+$Comp
+L Diode:1N4001 D1
+U 1 1 5CE7B69A
+P 4250 2650
+F 0 "D1" H 4250 2434 50  0000 C CNN
+F 1 "1N4001" H 4250 2525 50  0000 C CNN
+F 2 "Diode_THT:D_DO-41_SOD81_P10.16mm_Horizontal" H 4250 2475 50  0001 C CNN
+F 3 "http://www.vishay.com/docs/88503/1n4001.pdf" H 4250 2650 50  0001 C CNN
+	1    4250 2650
+	-1   0    0    1
+$EndComp
+Connection ~ 4400 2650
+Wire Wire Line
+	5500 4000 5700 4000
+$Comp
+L Diode:1N4001 D2
+U 1 1 5CE80A0F
+P 5700 4150
+F 0 "D2" V 5654 4229 50  0000 L CNN
+F 1 "1N4001" V 5745 4229 50  0000 L CNN
+F 2 "Diode_THT:D_DO-41_SOD81_P10.16mm_Horizontal" H 5700 3975 50  0001 C CNN
+F 3 "http://www.vishay.com/docs/88503/1n4001.pdf" H 5700 4150 50  0001 C CNN
+	1    5700 4150
+	0    1    1    0
+$EndComp
+Connection ~ 5700 4000
+Wire Wire Line
+	5700 4000 6000 4000
 $EndSCHEMATC

Commit message: change wiring to make layout easier
Changed lines of the file:
@@
 Wire Wire Line
 	8150 3700 8000 3700
-Wire Wire Line
-	6400 5150 7150 5150
-Wire Wire Line
-	7150 5150 7150 3800
-Wire Wire Line
-	7150 3800 7200 3800
-Wire Wire Line
-	5850 3400 6100 3400
-Wire Wire Line
-	6100 3400 6100 3700
-Wire Wire Line
-	6100 3700 7200 3700
-Wire Wire Line
-	7200 3600 6050 3600
-Wire Wire Line
-	6050 3600 6050 3500
-Wire Wire Line
-	6050 3500 5850 3500
-Wire Wire Line
-	7200 3400 7100 3400
-Wire Wire Line
-	7100 3400 7100 5350
-Wire Wire Line
-	7100 5350 6400 5350
 $Comp
 L power:+5V #PWR0112
@@
 Wire Wire Line
 	5700 4000 6000 4000
+Wire Wire Line
+	6400 5150 7050 5150
+Wire Wire Line
+	7050 5150 7050 3400
+Wire Wire Line
+	7050 3400 7200 3400
+Wire Wire Line
+	6400 5350 7100 5350
+Wire Wire Line
+	7100 5350 7100 3800
+Wire Wire Line
+	7100 3800 7200 3800
+Wire Wire Line
+	5850 3500 6050 3500
+Wire Wire Line
+	6050 3500 6050 3700
+Wire Wire Line
+	6050 3700 7200 3700
+Wire Wire Line
+	5850 3400 6100 3400
+Wire Wire Line
+	6100 3400 6100 3600
+Wire Wire Line
+	6100 3600 7200 3600
 $EndSCHEMATC

Commit message: add barrel jack and layout pcb again
Parts:
- added J2: Barrel_Jack_Switch, Connector_BarrelJack:BarrelJack_CUI_PJ-102AH_Horizontal, symbol Connector:Barrel_Jack_Switch
- renumbered J2 to J4, J4 to J5, J5 to J6, U3 to U2
Connections:
- wire segments 69 -> 75
Changed lines of the file:
@@
 encoding utf-8
 Sheet 1 1
-Title ""
-Date ""
-Rev ""
-Comp ""
+Title "PSU"
+Date "2019-05-26"
+Rev "1.0"
+Comp "Stephen Crane"
 Comment1 ""
 Comment2 ""
@@
 $EndDescr
 $Comp
-L power:GND #PWR0101
+L power:GND #PWR02
 U 1 1 5CD91970
 P 2250 3300
-F 0 "#PWR0101" H 2250 3050 50  0001 C CNN
+F 0 "#PWR02" H 2250 3050 50  0001 C CNN
 F 1 "GND" H 2255 3127 50  0000 C CNN
 F 2 "" H 2250 3300 50  0001 C CNN
@@
 $EndComp
 $Comp
-L power:+15V #PWR0102
+L power:+15V #PWR01
 U 1 1 5CD91A4B
 P 2250 2650
-F 0 "#PWR0102" H 2250 2500 50  0001 C CNN
+F 0 "#PWR01" H 2250 2500 50  0001 C CNN
 F 1 "+15V" H 2265 2823 50  0000 C CNN
 F 2 "" H 2250 2650 50  0001 C CNN
@@
 $EndComp
 $Comp
-L power:+5V #PWR0103
+L power:+5V #PWR05
 U 1 1 5CD91CC6
 P 4550 2650
-F 0 "#PWR0103" H 4550 2500 50  0001 C CNN
+F 0 "#PWR05" H 4550 2500 50  0001 C CNN
 F 1 "+5V" H 4565 2823 50  0000 C CNN
 F 2 "" H 4550 2650 50  0001 C CNN
@@
 	2700 3300 3400 3300
 $Comp
-L X9C103P:X9C103P U3
+L X9C103P:X9C103P U2
 U 1 1 5CD92F9E
 P 5700 5150
-F 0 "U3" H 5700 5720 50  0000 C CNN
+F 0 "U2" H 5700 5720 50  0000 C CNN
 F 1 "X9C103P" H 5700 5629 50  0000 C CNN
 F 2 "X9C103P:DIP254P762X533-8" H 5700 5150 50  0001 L BNN
@@
 $EndComp
 $Comp
-L power:GND #PWR0104
+L power:GND #PWR06
 U 1 1 5CD9328B
 P 4800 5650
-F 0 "#PWR0104" H 4800 5400 50  0001 C CNN
+F 0 "#PWR06" H 4800 5400 50  0001 C CNN
 F 1 "GND" H 4805 5477 50  0000 C CNN
 F 2 "" H 4800 5650 50  0001 C CNN
@@
 $EndComp
 $Comp
-L power:GND #PWR0105
+L power:GND #PWR011
 U 1 1 5CD93910
 P 6400 5650
-F 0 "#PWR0105" H 6400 5400 50  0001 C CNN
+F 0 "#PWR011" H 6400 5400 50  0001 C CNN
 F 1 "GND" H 6405 5477 50  0000 C CNN
 F 2 "" H 6400 5650 50  0001 C CNN
@@
 $EndComp
 $Comp
-L power:+5V #PWR0106
+L power:+5V #PWR010
 U 1 1 5CD93966
 P 6400 4800
-F 0 "#PWR0106" H 6400 4650 50  0001 C CNN
+F 0 "#PWR010" H 6400 4650 50  0001 C CNN
 F 1 "+5V" H 6415 4973 50  0000 C CNN
 F 2 "" H 6400 4800 50  0001 C CNN
@@
 $EndComp
 $Comp
-L power:+15V #PWR0107
+L power:+15V #PWR03
 U 1 1 5CD98A23
 P 2650 4150
-F 0 "#PWR0107" H 2650 4000 50  0001 C CNN
+F 0 "#PWR03" H 2650 4000 50  0001 C CNN
 F 1 "+15V" H 2665 4323 50  0000 C CNN
 F 2 "" H 2650 4150 50  0001 C CNN
@@
 $EndComp
 $Comp
-L power:GND #PWR0108
+L power:GND #PWR04
 U 1 1 5CD98A46
 P 2650 4250
-F 0 "#PWR0108" H 2650 4000 50  0001 C CNN
+F 0 "#PWR04" H 2650 4000 50  0001 C CNN
 F 1 "GND" H 2655 4077 50  0000 C CNN
 F 2 "" H 2650 4250 50  0001 C CNN
@@
 $EndComp
 $Comp
-L Connector:Conn_01x06_Male J2
+L Connector:Conn_01x06_Male J4
 U 1 1 5CD99276
 P 5650 3400
-F 0 "J2" H 5756 3778 50  0000 C CNN
+F 0 "J4" H 5756 3778 50  0000 C CNN
 F 1 "INA219 breakout" H 5756 3687 50  0000 C CNN
 F 2 "Connector_PinHeader_2.54mm:PinHeader_1x06_P2.54mm_Vertical" H 5650 3400 50  0001 C CNN
@@
 $EndComp
 $Comp
-L power:+5V #PWR0109
+L power:+5V #PWR08
 U 1 1 5CD992DC
 P 6200 3150
-F 0 "#PWR0109" H 6200 3000 50  0001 C CNN
+F 0 "#PWR08" H 6200 3000 50  0001 C CNN
 F 1 "+5V" H 6215 3323 50  0000 C CNN
 F 2 "" H 6200 3150 50  0001 C CNN
@@
 $EndComp
 $Comp
-L power:GND #PWR0110
+L power:GND #PWR09
 U 1 1 5CD99302
 P 6200 3350
-F 0 "#PWR0110" H 6200 3100 50  0001 C CNN
+F 0 "#PWR09" H 6200 3100 50  0001 C CNN
 F 1 "GND" H 6205 3177 50  0000 C CNN
 F 2 "" H 6200 3350 50  0001 C CNN
@@
 $EndComp
 $Comp
-L power:GND #PWR0111
+L power:GND #PWR07
 U 1 1 5CD9960B
 P 6000 4350
-F 0 "#PWR0111" H 6000 4100 50  0001 C CNN
+F 0 "#PWR07" H 6000 4100 50  0001 C CNN
 F 1 "GND" H 6005 4177 50  0000 C CNN
 F 2 "" H 6000 4350 50  0001 C CNN
@@
 	5950 3600 5850 3600
 $Comp
-L Connector:Conn_01x08_Female J4
+L Connector:Conn_01x08_Female J5
 U 1 1 5CD9B59C
 P 7400 3500
-F 0 "J4" H 7428 3476 50  0000 L CNN
+F 0 "J5" H 7428 3476 50  0000 L CNN
 F 1 "WWG-A" H 7428 3385 50  0000 L CNN
 F 2 "Connector_PinHeader_2.54mm:PinHeader_1x08_P2.54mm_Vertical" H 7400 3500 50  0001 C CNN
@@
 $EndComp
 $Comp
-L Connector:Conn_01x08_Female J5
+L Connector:Conn_01x08_Female J6
 U 1 1 5CD9B613
 P 7800 3500
-F 0 "J5" H 7694 3985 50  0000 C CNN
+F 0 "J6" H 7694 3985 50  0000 C CNN
 F 1 "WWG-B" H 7694 3894 50  0000 C CNN
 F 2 "Connector_PinHeader_2.54mm:PinHeader_1x08_P2.54mm_Vertical" H 7800 3500 50  0001 C CNN
@@
 	8150 3700 8000 3700
 $Comp
-L power:+5V #PWR0112
+L power:+5V #PWR013
 U 1 1 5CD9E06C
 P 7150 3150
-F 0 "#PWR0112" H 7150 3000 50  0001 C CNN
+F 0 "#PWR013" H 7150 3000 50  0001 C CNN
 F 1 "+5V" H 7165 3323 50  0000 C CNN
 F 2 "" H 7150 3150 50  0001 C CNN
@@
 $EndComp
 $Comp
-L power:GND #PWR0113
+L power:GND #PWR012
 U 1 1 5CD9E09B
 P 6950 3350
-F 0 "#PWR0113" H 6950 3100 50  0001 C CNN
+F 0 "#PWR012" H 6950 3100 50  0001 C CNN
 F 1 "GND" H 6955 3177 50  0000 C CNN
 F 2 "" H 6950 3350 50  0001 C CNN
@@
 	4650 4450 4650 5150
 $Comp
-L power:PWR_FLAG #FLG0101
+L power:PWR_FLAG #FLG03
 U 1 1 5CE68781
 P 4400 2650
-F 0 "#FLG0101" H 4400 2725 50  0001 C CNN
+F 0 "#FLG03" H 4400 2725 50  0001 C CNN
 F 1 "PWR_FLAG" H 4400 2824 50  0001 C CNN
 F 2 "" H 4400 2650 50  0001 C CNN
@@
 	2500 4250 2650 4250
 $Comp
-L power:PWR_FLAG #FLG0102
+L power:PWR_FLAG #FLG01
 U 1 1 5CE6B5B3
 P 2500 4150
-F 0 "#FLG0102" H 2500 4225 50  0001 C CNN
+F 0 "#FLG01" H 2500 4225 50  0001 C CNN
 F 1 "PWR_FLAG" H 2500 4324 50  0001 C CNN
 F 2 "" H 2500 4150 50  0001 C CNN
@@
 Connection ~ 2500 4150
 $Comp
-L power:PWR_FLAG #FLG0103
+L power:PWR_FLAG #FLG02
 U 1 1 5CE6B602
 P 2500 4250
-F 0 "#FLG0103" H 2500 4325 50  0001 C CNN
+F 0 "#FLG02" H 2500 4325 50  0001 C CNN
 F 1 "PWR_FLAG" H 2500 4423 50  0001 C CNN
 F 2 "" H 2500 4250 50  0001 C CNN
@@
 	5850 3500 6050 3500
 Wire Wire Line
-	6050 3500 6050 3700
-Wire Wire Line
-	6050 3700 7200 3700
-Wire Wire Line
 	5850 3400 6100 3400
-Wire Wire Line
-	6100 3400 6100 3600
-Wire Wire Line
-	6100 3600 7200 3600
+$Comp
+L Connector:Barrel_Jack_Switch J2
+U 1 1 5CEA7F8F
+P 2450 4850
+F 0 "J2" H 2220 4800 50  0000 R CNN
+F 1 "Barrel_Jack_Switch" H 2220 4891 50  0000 R CNN
+F 2 "Connector_BarrelJack:BarrelJack_CUI_PJ-102AH_Horizontal" H 2500 4810 50  0001 C CNN
+F 3 "~" H 2500 4810 50  0001 C CNN
+	1    2450 4850
+	1    0    0    1
+$EndComp
+Wire Wire Line
+	2650 4250 2750 4250
+Wire Wire Line
+	2750 4250 2750 4750
+Connection ~ 2650 4250
+Wire Wire Line
+	2750 4750 2750 4850
+Connection ~ 2750 4750
+Wire Wire Line
+	2750 4950 2850 4950
+Wire Wire Line
+	2850 4950 2850 4150
+Wire Wire Line
+	2850 4150 2650 4150
+Connection ~ 2650 4150
+Wire Wire Line
+	6100 3400 6100 3700
+Wire Wire Line
+	6100 3700 7200 3700
+Wire Wire Line
+	6050 3500 6050 3600
+Wire Wire Line
+	6050 3600 7200 3600
 $EndSCHEMATC

Commit message: layout again
Parts:
- removed D1: 1N4001, Diode_THT:D_DO-41_SOD81_P10.16mm_Horizontal, symbol Diode:1N4001
Changed lines of the file:
@@
 	7150 3200 7200 3200
-Wire Wire Line
-	3900 2650 4100 2650
 Wire Wire Line
 	4400 2650 4550 2650
@@
 NoConn ~ 7200 3500
 NoConn ~ 5000 5050
-$Comp
-L Diode:1N4001 D1
-U 1 1 5CE7B69A
-P 4250 2650
-F 0 "D1" H 4250 2434 50  0000 C CNN
-F 1 "1N4001" H 4250 2525 50  0000 C CNN
-F 2 "Diode_THT:D_DO-41_SOD81_P10.16mm_Horizontal" H 4250 2475 50  0001 C CNN
-F 3 "http://www.vishay.com/docs/88503/1n4001.pdf" H 4250 2650 50  0001 C CNN
-	1    4250 2650
-	-1   0    0    1
-$EndComp
-Connection ~ 4400 2650
 Wire Wire Line
 	5500 4000 5700 4000
@@
 Wire Wire Line
 	6050 3600 7200 3600
+Wire Wire Line
+	3900 2650 4400 2650
+Connection ~ 4400 2650
 $EndSCHEMATC
